Commit message: remove cob4-2 leftover

File: cob4-2/calibration/calibration_offset.urdf.xacro (robot description, xacro)
@@ -49,32 +49,4 @@
 	<xacro:property name="offset_sensorring_pitch" value="0.0"/>
 	<xacro:property name="offset_sensorring_yaw" value="0.0"/>
-	<!-- arm right mount positions | relative to torso_3_link -->
-	<xacro:property name="offset_arm_right_x" value="0.0"/>
-	<xacro:property name="offset_arm_right_y" value="0.0"/>
-	<xacro:property name="offset_arm_right_z" value="0.0"/>
-	<xacro:property name="offset_arm_right_roll" value="0.0"/>
-	<xacro:property name="offset_arm_right_pitch" value="0.0"/>
-	<xacro:property name="offset_arm_right_yaw" value="0.0"/>
-	<!-- arm left mount positions | relative to torso_3_link -->
-	<xacro:property name="offset_arm_left_x" value="0.0"/>
-	<xacro:property name="offset_arm_left_y" value="0.0"/>
-	<xacro:property name="offset_arm_left_z" value="0.0"/>
-	<xacro:property name="offset_arm_left_roll" value="0.0"/>
-	<xacro:property name="offset_arm_left_pitch" value="0.0"/>
-	<xacro:property name="offset_arm_left_yaw" value="0.0"/>
-	<!-- gripper right mount positions | relative to arm_right_7_link -->
-	<xacro:property name="offset_gripper_right_x" value="0.0"/>
-	<xacro:property name="offset_gripper_right_y" value="0.0"/>
-	<xacro:property name="offset_gripper_right_z" value="0.0"/>
-	<xacro:property name="offset_gripper_right_roll" value="0.0"/>
-	<xacro:property name="offset_gripper_right_pitch" value="0.0"/>
-	<xacro:property name="offset_gripper_right_yaw" value="0.0"/>
-	<!-- gripper left mount positions | relative to arm_left_7_link -->
-	<xacro:property name="offset_gripper_left_x" value="0.0"/>
-	<xacro:property name="offset_gripper_left_y" value="0.0"/>
-	<xacro:property name="offset_gripper_left_z" value="0.0"/>
-	<xacro:property name="offset_gripper_left_roll" value="0.0"/>
-	<xacro:property name="offset_gripper_left_pitch" value="0.0"/>
-	<xacro:property name="offset_gripper_left_yaw" value="0.0"/>
 	<!-- *********************************** -->
 	<!-- kinematic chain reference positions -->
