Commit message: renamed sensorring camera

File: cob4-8/calibration/calibration_offset.urdf.xacro (robot description, xacro)
@@ -103,17 +103,10 @@
 	<xacro:property name="offset_torso_cam3d_down_yaw" value="0.0"/>
 	<!-- cam3d | handeye calibration | relative to sensorring_link -->
-	<xacro:property name="offset_sensorring_cam3d_front_x" value="0.0"/>
-	<xacro:property name="offset_sensorring_cam3d_front_y" value="0.0"/>
-	<xacro:property name="offset_sensorring_cam3d_front_z" value="0.0"/>
-	<xacro:property name="offset_sensorring_cam3d_front_roll" value="0.0"/>
-	<xacro:property name="offset_sensorring_cam3d_front_pitch" value="0.0"/>
-	<xacro:property name="offset_sensorring_cam3d_front_yaw" value="0.0"/>
-	<!-- cam3d | handeye calibration | relative to sensorring_link -->
-	<xacro:property name="offset_sensorring_cam3d_back_x" value="0.0"/>
-	<xacro:property name="offset_sensorring_cam3d_back_y" value="0.0"/>
-	<xacro:property name="offset_sensorring_cam3d_back_z" value="0.0"/>
-	<xacro:property name="offset_sensorring_cam3d_back_roll" value="0.0"/>
-	<xacro:property name="offset_sensorring_cam3d_back_pitch" value="0.0"/>
-	<xacro:property name="offset_sensorring_cam3d_back_yaw" value="0.0"/>
+	<xacro:property name="offset_sensorring_cam3d_x" value="0.0"/>
+	<xacro:property name="offset_sensorring_cam3d_y" value="0.0"/>
+	<xacro:property name="offset_sensorring_cam3d_z" value="0.0"/>
+	<xacro:property name="offset_sensorring_cam3d_roll" value="0.0"/>
+	<xacro:property name="offset_sensorring_cam3d_pitch" value="0.0"/>
+	<xacro:property name="offset_sensorring_cam3d_yaw" value="0.0"/>
 	<!-- cam | handeye calibration | relative to head_3_link -->
 	<xacro:property name="offset_head_cam_x" value="0.0"/>
