Commit message: full config for cob4-10 tlabs

File: cob4-10/calibration/calibration_offset.urdf.xacro (robot description, xacro)
@@ -25,3 +25,94 @@
 	<xacro:property name="offset_laser_right_pitch" value="0.0"/>
 	<xacro:property name="offset_laser_right_yaw" value="0.0"/>
+	<!-- *********************** -->
+	<!-- upper robot calibration -->
+	<!-- *********************** -->
+	<!-- torso mount positions | relative to base_link -->
+	<xacro:property name="offset_torso_x" value="0.0"/>
+	<xacro:property name="offset_torso_y" value="0.0"/>
+	<xacro:property name="offset_torso_z" value="0.0"/>
+	<xacro:property name="offset_torso_roll" value="0.0"/>
+	<xacro:property name="offset_torso_pitch" value="0.0"/>
+	<xacro:property name="offset_torso_yaw" value="0.0"/>
+	<!-- head mount positions | relative to torso_3_link -->
+	<xacro:property name="offset_head_x" value="0.0"/>
+	<xacro:property name="offset_head_y" value="0.0"/>
+	<xacro:property name="offset_head_z" value="0.0"/>
+	<xacro:property name="offset_head_roll" value="0.0"/>
+	<xacro:property name="offset_head_pitch" value="0.0"/>
+	<xacro:property name="offset_head_yaw" value="0.0"/>
+	<!-- sersorring mount positions | relative to head_3_link -->
+	<xacro:property name="offset_sensorring_x" value="0.0"/>
+	<xacro:property name="offset_sensorring_y" value="0.0"/>
+	<xacro:property name="offset_sensorring_z" value="0.0"/>
+	<xacro:property name="offset_sensorring_roll" value="0.0"/>
+	<xacro:property name="offset_sensorring_pitch" value="0.0"/>
+	<xacro:property name="offset_sensorring_yaw" value="0.0"/>
+	<!-- arm right mount positions | relative to torso_3_link -->
+	<xacro:property name="offset_arm_right_x" value="0.0"/>
+	<xacro:property name="offset_arm_right_y" value="0.0"/>
+	<xacro:property name="offset_arm_right_z" value="0.0"/>
+	<xacro:property name="offset_arm_right_roll" value="0.0"/>
+	<xacro:property name="offset_arm_right_pitch" value="0.0"/>
+	<xacro:property name="offset_arm_right_yaw" value="0.0"/>
+	<!-- arm left mount positions | relative to torso_3_link -->
+	<xacro:property name="offset_arm_left_x" value="0.0"/>
+	<xacro:property name="offset_arm_left_y" value="0.0"/>
+	<xacro:property name="offset_arm_left_z" value="0.0"/>
+	<xacro:property name="offset_arm_left_roll" value="0.0"/>
+	<xacro:property name="offset_arm_left_pitch" value="0.0"/>
+	<xacro:property name="offset_arm_left_yaw" value="0.0"/>
+	<!-- gripper right mount positions | relative to arm_7_link -->
+	<xacro:property name="offset_gripper_right_x" value="0.0"/>
+	<xacro:property name="offset_gripper_right_y" value="0.0"/>
+	<xacro:property name="offset_gripper_right_z" value="0.0"/>
+	<xacro:property name="offset_gripper_right_roll" value="0.0"/>
+	<xacro:property name="offset_gripper_right_pitch" value="0.0"/>
+	<xacro:property name="offset_gripper_right_yaw" value="0.0"/>
+	<!-- gripper left mount positions | relative to arm_7_link -->
+	<xacro:property name="offset_gripper_left_x" value="0.0"/>
+	<xacro:property name="offset_gripper_left_y" value="0.0"/>
+	<xacro:property name="offset_gripper_left_z" value="0.0"/>
+	<xacro:property name="offset_gripper_left_roll" value="0.0"/>
+	<xacro:property name="offset_gripper_left_pitch" value="0.0"/>
+	<xacro:property name="offset_gripper_left_yaw" value="0.0"/>
+	<!-- *********************************** -->
+	<!-- kinematic chain reference positions -->
+	<!-- *********************************** -->
+	<!-- this feature is no longer supported as urdfdom does not parse the according 'calibration_rising' tag -->
+	<!-- cam3d left | handeye calibration | relative to torso_3_link -->
+	<xacro:property name="offset_torso_cam3d_left_x" value="0.0"/>
+	<xacro:property name="offset_torso_cam3d_left_y" value="0.0"/>
+	<xacro:property name="offset_torso_cam3d_left_z" value="0.0"/>
+	<xacro:property name="offset_torso_cam3d_left_roll" value="0.0"/>
+	<xacro:property name="offset_torso_cam3d_left_pitch" value="0.0"/>
+	<xacro:property name="offset_torso_cam3d_left_yaw" value="0.0"/>
+	<!-- cam3d right | handeye calibration | relative to torso_3_link -->
+	<xacro:property name="offset_torso_cam3d_right_x" value="0.0"/>
+	<xacro:property name="offset_torso_cam3d_right_y" value="0.0"/>
+	<xacro:property name="offset_torso_cam3d_right_z" value="0.0"/>
+	<xacro:property name="offset_torso_cam3d_right_roll" value="0.0"/>
+	<xacro:property name="offset_torso_cam3d_right_pitch" value="0.0"/>
+	<xacro:property name="offset_torso_cam3d_right_yaw" value="0.0"/>
+	<!-- cam3d down | handeye calibration | relative to torso_3_link -->
+	<xacro:property name="offset_torso_cam3d_down_x" value="0.0"/>
+	<xacro:property name="offset_torso_cam3d_down_y" value="0.0"/>
+	<xacro:property name="offset_torso_cam3d_down_z" value="0.0"/>
+	<xacro:property name="offset_torso_cam3d_down_roll" value="0.0"/>
+	<xacro:property name="offset_torso_cam3d_down_pitch" value="0.0"/>
+	<xacro:property name="offset_torso_cam3d_down_yaw" value="0.0"/>
+	<!-- cam3d | handeye calibration | relative to sensorring_link -->
+	<xacro:property name="offset_sensorring_cam3d_x" value="0.0"/>
+	<xacro:property name="offset_sensorring_cam3d_y" value="0.0"/>
+	<xacro:property name="offset_sensorring_cam3d_z" value="0.0"/>
+	<xacro:property name="offset_sensorring_cam3d_roll" value="0.0"/>
+	<xacro:property name="offset_sensorring_cam3d_pitch" value="0.0"/>
+	<xacro:property name="offset_sensorring_cam3d_yaw" value="0.0"/>
+	<!-- cam | handeye calibration | relative to head_3_link -->
+	<xacro:property name="offset_head_cam_x" value="0.0"/>
+	<xacro:property name="offset_head_cam_y" value="0.0"/>
+	<xacro:property name="offset_head_cam_z" value="0.0"/>
+	<xacro:property name="offset_head_cam_roll" value="0.0"/>
+	<xacro:property name="offset_head_cam_pitch" value="0.0"/>
+	<xacro:property name="offset_head_cam_yaw" value="0.0"/>
 </robot>

Commit message: setup cob4-10

File: cob4-10/calibration/calibration_offset.urdf.xacro (robot description, xacro)
@@ -103,10 +103,17 @@
 	<xacro:property name="offset_torso_cam3d_down_yaw" value="0.0"/>
 	<!-- cam3d | handeye calibration | relative to sensorring_link -->
-	<xacro:property name="offset_sensorring_cam3d_x" value="0.0"/>
-	<xacro:property name="offset_sensorring_cam3d_y" value="0.0"/>
-	<xacro:property name="offset_sensorring_cam3d_z" value="0.0"/>
-	<xacro:property name="offset_sensorring_cam3d_roll" value="0.0"/>
-	<xacro:property name="offset_sensorring_cam3d_pitch" value="0.0"/>
-	<xacro:property name="offset_sensorring_cam3d_yaw" value="0.0"/>
+	<xacro:property name="offset_sensorring_cam3d_front_x" value="0.0"/>
+	<xacro:property name="offset_sensorring_cam3d_front_y" value="0.0"/>
+	<xacro:property name="offset_sensorring_cam3d_front_z" value="0.0"/>
+	<xacro:property name="offset_sensorring_cam3d_front_roll" value="0.0"/>
+	<xacro:property name="offset_sensorring_cam3d_front_pitch" value="0.0"/>
+	<xacro:property name="offset_sensorring_cam3d_front_yaw" value="0.0"/>
+	<!-- cam3d | handeye calibration | relative to sensorring_link -->
+	<xacro:property name="offset_sensorring_cam3d_back_x" value="0.0"/>
+	<xacro:property name="offset_sensorring_cam3d_back_y" value="0.0"/>
+	<xacro:property name="offset_sensorring_cam3d_back_z" value="0.0"/>
+	<xacro:property name="offset_sensorring_cam3d_back_roll" value="0.0"/>
+	<xacro:property name="offset_sensorring_cam3d_back_pitch" value="0.0"/>
+	<xacro:property name="offset_sensorring_cam3d_back_yaw" value="0.0"/>
 	<!-- cam | handeye calibration | relative to head_3_link -->
 	<xacro:property name="offset_head_cam_x" value="0.0"/>
