Commit message: update cob4-7 setup , cob4-paul-stuttgart

File: cob4-7/calibration/calibration_offset.urdf.xacro (robot description, xacro)
@@ -49,18 +49,4 @@
 	<xacro:property name="offset_sensorring_pitch" value="0.0"/>
 	<xacro:property name="offset_sensorring_yaw" value="0.0"/>
-	<!-- arm right mount positions | relative to torso_3_link -->
-	<xacro:property name="offset_arm_right_x" value="0.0"/>
-	<xacro:property name="offset_arm_right_y" value="0.0"/>
-	<xacro:property name="offset_arm_right_z" value="0.0"/>
-	<xacro:property name="offset_arm_right_roll" value="0.0"/>
-	<xacro:property name="offset_arm_right_pitch" value="0.0"/>
-	<xacro:property name="offset_arm_right_yaw" value="0.0"/>
-	<!-- arm left mount positions | relative to torso_3_link -->
-	<xacro:property name="offset_arm_left_x" value="0.0"/>
-	<xacro:property name="offset_arm_left_y" value="0.0"/>
-	<xacro:property name="offset_arm_left_z" value="0.0"/>
-	<xacro:property name="offset_arm_left_roll" value="0.0"/>
-	<xacro:property name="offset_arm_left_pitch" value="0.0"/>
-	<xacro:property name="offset_arm_left_yaw" value="0.0"/>
 	<!-- *********************************** -->
 	<!-- kinematic chain reference positions -->

Commit message: use zr300 for torso_right camera

File: cob4-7/calibration/calibration_offset.urdf.xacro (robot description, xacro)
@@ -74,4 +74,11 @@
 	<xacro:property name="offset_torso_cam3d_down_pitch" value="0.0"/>
 	<xacro:property name="offset_torso_cam3d_down_yaw" value="0.0"/>
+	<!-- cam3d down | handeye calibration | relative to torso_3_link -->
+	<xacro:property name="offset_torso_cam3d_zr300_x" value="0.0"/>
+	<xacro:property name="offset_torso_cam3d_zr300_y" value="0.0"/>
+	<xacro:property name="offset_torso_cam3d_zr300_z" value="0.0"/>
+	<xacro:property name="offset_torso_cam3d_zr300_roll" value="0.0"/>
+	<xacro:property name="offset_torso_cam3d_zr300_pitch" value="0.0"/>
+	<xacro:property name="offset_torso_cam3d_zr300_yaw" value="0.0"/>
 	<!-- cam3d | handeye calibration | relative to sensorring_link -->
 	<xacro:property name="offset_sensorring_cam3d_x" value="0.0"/>

Commit message: finalize zr300 transformations

File: cob4-7/calibration/calibration_offset.urdf.xacro (robot description, xacro)
@@ -74,11 +74,4 @@
 	<xacro:property name="offset_torso_cam3d_down_pitch" value="0.0"/>
 	<xacro:property name="offset_torso_cam3d_down_yaw" value="0.0"/>
-	<!-- cam3d down | handeye calibration | relative to torso_3_link -->
-	<xacro:property name="offset_torso_cam3d_zr300_x" value="0.0"/>
-	<xacro:property name="offset_torso_cam3d_zr300_y" value="0.0"/>
-	<xacro:property name="offset_torso_cam3d_zr300_z" value="0.0"/>
-	<xacro:property name="offset_torso_cam3d_zr300_roll" value="0.0"/>
-	<xacro:property name="offset_torso_cam3d_zr300_pitch" value="0.0"/>
-	<xacro:property name="offset_torso_cam3d_zr300_yaw" value="0.0"/>
 	<!-- cam3d | handeye calibration | relative to sensorring_link -->
 	<xacro:property name="offset_sensorring_cam3d_x" value="0.0"/>

Commit message: setup cob4-7

File: cob4-7/calibration/calibration_offset.urdf.xacro (robot description, xacro)
@@ -49,4 +49,32 @@
 	<xacro:property name="offset_sensorring_pitch" value="0.0"/>
 	<xacro:property name="offset_sensorring_yaw" value="0.0"/>
+	<!-- arm right mount positions | relative to torso_3_link -->
+	<xacro:property name="offset_arm_right_x" value="0.0"/>
+	<xacro:property name="offset_arm_right_y" value="0.0"/>
+	<xacro:property name="offset_arm_right_z" value="0.0"/>
+	<xacro:property name="offset_arm_right_roll" value="0.0"/>
+	<xacro:property name="offset_arm_right_pitch" value="0.0"/>
+	<xacro:property name="offset_arm_right_yaw" value="0.0"/>
+	<!-- arm left mount positions | relative to torso_3_link -->
+	<xacro:property name="offset_arm_left_x" value="0.0"/>
+	<xacro:property name="offset_arm_left_y" value="0.0"/>
+	<xacro:property name="offset_arm_left_z" value="0.0"/>
+	<xacro:property name="offset_arm_left_roll" value="0.0"/>
+	<xacro:property name="offset_arm_left_pitch" value="0.0"/>
+	<xacro:property name="offset_arm_left_yaw" value="0.0"/>
+	<!-- gripper right mount positions | relative to arm_7_link -->
+	<xacro:property name="offset_gripper_right_x" value="0.0"/>
+	<xacro:property name="offset_gripper_right_y" value="0.0"/>
+	<xacro:property name="offset_gripper_right_z" value="0.0"/>
+	<xacro:property name="offset_gripper_right_roll" value="0.0"/>
+	<xacro:property name="offset_gripper_right_pitch" value="0.0"/>
+	<xacro:property name="offset_gripper_right_yaw" value="0.0"/>
+	<!-- gripper left mount positions | relative to arm_7_link -->
+	<xacro:property name="offset_gripper_left_x" value="0.0"/>
+	<xacro:property name="offset_gripper_left_y" value="0.0"/>
+	<xacro:property name="offset_gripper_left_z" value="0.0"/>
+	<xacro:property name="offset_gripper_left_roll" value="0.0"/>
+	<xacro:property name="offset_gripper_left_pitch" value="0.0"/>
+	<xacro:property name="offset_gripper_left_yaw" value="0.0"/>
 	<!-- *********************************** -->
 	<!-- kinematic chain reference positions -->
