Commit message: fixup cob4-25 for noetic

File: cob4-25/calibration/calibration_offset.urdf.xacro (robot description, xacro)
@@ -49,4 +49,18 @@
 	<xacro:property name="offset_sensorring_pitch" value="0.0"/>
 	<xacro:property name="offset_sensorring_yaw" value="0.0"/>
+	<!-- arm right mount positions | relative to torso_3_link -->
+	<xacro:property name="offset_arm_right_x" value="0.0"/>
+	<xacro:property name="offset_arm_right_y" value="0.0"/>
+	<xacro:property name="offset_arm_right_z" value="0.0"/>
+	<xacro:property name="offset_arm_right_roll" value="0.0"/>
+	<xacro:property name="offset_arm_right_pitch" value="0.0"/>
+	<xacro:property name="offset_arm_right_yaw" value="0.0"/>
+	<!-- arm left mount positions | relative to torso_3_link -->
+	<xacro:property name="offset_arm_left_x" value="0.0"/>
+	<xacro:property name="offset_arm_left_y" value="0.0"/>
+	<xacro:property name="offset_arm_left_z" value="0.0"/>
+	<xacro:property name="offset_arm_left_roll" value="0.0"/>
+	<xacro:property name="offset_arm_left_pitch" value="0.0"/>
+	<xacro:property name="offset_arm_left_yaw" value="0.0"/>
 	<!-- *********************************** -->
 	<!-- kinematic chain reference positions -->
